File: Hardware/Kicad/CAT FLAP/CatFlap_PCB/CatFlap_PCB/CatFlap_PCB.kicad_pcb (KiCad board)
At the start: 2 copper layers, 196 x 25 mm, 45 parts, among them J2 Conn_01x03, J3 Battery pack, J4 Conn_01x03_Socket, J5 Conn_ARM_SWD_TagConnect_TC203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, J6 Conn_01x02, J7 Conn_01x06, J8 Conn_01x20, J9 Conn_01x20, M1 Motor_DC, Q1 NX3008CBKS, Q2 Q_PMOS_DGS, SW1 SW_Push, SW2 SW_Push, SW3 SW_Push, SW4 SW_Push, T1 NX3008NBKS, T2 NX3008NBKS, U3 TPS62132

Commit message: Add files via upload
Parts:
- removed C16, C17: 1u, Capacitor_SMD:C_0603_1608Metric
- removed J7: Conn_01x06, Connector_PinHeader_2.54mm:PinHeader_1x06_P2.54mm_Vertical
- removed SW4: SW_Push, Button_Switch_SMD:SW_Push_1P1T_NO_Vertical_Wuerth_434133025816
- added C3: 1u, Capacitor_SMD:C_0603_1608Metric, F.Cu at (201.4, 79.4)
- added C4: 1u, Capacitor_SMD:C_0603_1608Metric, F.Cu at (186.2, 93.0)
- added D1: LED_RGB, LED_SMD:LED_RGB_PLCC-6, F.Cu at (78.3, 75.7)
- added J1: Conn_01x08, Connector_PinHeader_2.54mm:PinHeader_1x08_P2.54mm_Vertical, F.Cu at (220.5, 75.8)
- added JP2: SolderJumper_3_Bridged12, Jumper:SolderJumper-3_P1.3mm_Bridged12_RoundedPad1.0x1.5mm, F.Cu at (198.5, 79.4)
- added JP3: SolderJumper_3_Bridged12, Jumper:SolderJumper-3_P1.3mm_Bridged12_RoundedPad1.0x1.5mm, F.Cu at (189.1, 92.9)
- added JP4: SolderJumper_3_Bridged12, Jumper:SolderJumper-3_P1.3mm_Bridged12_RoundedPad1.0x1.5mm, F.Cu at (102.8, 88.8)
- added L1: 2.2u, Inductor_SMD:L_Coilcraft_XxL4020, F.Cu at (116.2, 88.8)
- added R1: 6.8, Resistor_SMD:R_0603_1608Metric, F.Cu at (195.2, 87.5)
- added R10: 0, Resistor_SMD:R_0603_1608Metric, F.Cu at (108.0, 77.0)
- added R14: 0, Resistor_SMD:R_0603_1608Metric, F.Cu at (120.3, 90.3)
- added R2: 6.8, Resistor_SMD:R_0603_1608Metric, F.Cu at (199.8, 83.3)
- added T3: NX3008NBKS, Package_TO_SOT_SMD:SOT-363_SC-70-6, F.Cu at (195.8, 84.4)
- added U2: DRV8837DSGR, DRV8837DSGR:SON50P200X200X80-9N, F.Cu at (99.5, 90.0)
- C12, C15: footprint Capacitor_SMD:C_0603_1608Metric -> Capacitor_SMD:C_1210_3225Metric
- C18, C21: footprint Capacitor_SMD:C_0603_1608Metric -> Capacitor_SMD:C_0805_2012Metric
- J3: footprint Connector_JST:JST_XH_B2B-XH-A_1x02_P2.50mm_Vertical -> Battery:BatteryHolder_MPD_BH-18650-PC2
- J5: value Conn_ARM_SWD_TagConnect_TC2030-NL -> Conn_01x03; footprint Connector:Tag-Connect_TC2030-IDC-NL_2x03_P1.27mm_Vertical -> Connector_PinHeader_2.54mm:PinHeader_1x03_P2.54mm_Vertical
- R11, R12: value 100 -> 6.8
- R4: value 20 -> 22
- SW3: footprint Button_Switch_SMD:SW_Push_1P1T_NO_6x6mm_H9.5mm -> Button_Switch_SMD:SW_Push_1P1T_NO_Vertical_Wuerth_434133025816
- moved R5 184.9 mm to (83.0, 77.2), turned to 180 degrees
- moved R4 184.6 mm to (83.0, 75.7), turned to 180 degrees
- moved R3 184.4 mm to (83.0, 74.0), turned to 180 degrees
- moved T1 178.4 mm to (88.2, 74.7)
- moved T2 177.9 mm to (88.2, 77.8), turned to 180 degrees
- moved J3 174.2 mm to (203.3, 75.4), turned to -90 degrees
- moved C15 162.8 mm to (95.9, 86.6), turned to -90 degrees
- moved C13 159.0 mm to (98.5, 87.1), turned to -90 degrees
- moved C14 157.7 mm to (100.4, 87.1), turned to -90 degrees
- moved D5 146.7 mm to (102.1, 76.8), turned to 90 degrees
- moved M1 140.9 mm to (90.7, 92.8), turned to -90 degrees
- moved J2 138.5 mm to (95.0, 93.2), turned to 90 degrees
- moved D4 123.6 mm to (119.3, 93.0), turned to -90 degrees
- moved J5 101.9 mm to (188.4, 81.0), turned to 0 degrees
- moved F1 90.5 mm to (120.3, 74.8)
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Connections:
- C12 pad 2: Net-(Q2-S) -> VDD
- D4 pad 2: IR_R_INSIDE -> Net-(D4-A)
- D5 pad 2: IR_R_OUTSIDE -> Net-(D5-A)
- F1 pad 2: Net-(Q2-S) -> VDD
- J3 pad 2: VDD -> Net-(J3-V+)
- J5 pad 1: +3.3V -> Antenn_Analog
- J5 pad 2: SWDIO -> /GP27_A0
- J5 pad 3: Reset -> BAT_MON
- J6 pad 1: VDD -> Net-(J3-V+)
- J8 pad 11: /RUN -> Reset
- J8 pad 19: /GP17 -> Antenn_Digital_2
- J8 pad 20: /GP16 -> Antenn_Digital_1
- J8 pad 6: /ADC_VREF -> ADC_VREF_Antenn
- J8 pad 7: BAT_MON -> IR_R_OUTSIDE
- J8 pad 9: /GP27_A1 -> IR_R_INSIDE
- J9 pad 10: /GP7 -> IR_T_OUTSIDE
- J9 pad 11: /GP8 -> IR_T_INSIDE
- J9 pad 2: /GP1 -> M_SLEEP
- J9 pad 4: /GP2 -> LED_B
- J9 pad 5: /GP3 -> LED_G
- J9 pad 6: /GP4 -> LED_R
- J9 pad 7: /GP5 -> M_UNLOCK
- J9 pad 9: /GP6 -> M_LOCK
- Q2 pad 1: VDD -> Net-(J3-V+)
- Q2 pad 3: Net-(Q2-S) -> VDD
Routing:
- net +3.3V: track 3.75 -> 280.1 mm, vias 0 -> 4
- net Net-(J3-V+): track 0.00 -> 178.6 mm, vias 0 -> 3
- net VDD: track 23.1 -> 178.0 mm, vias 0 -> 8
- net ADC_VREF_Antenn: track 0.00 -> 85.0 mm
- net LED_R: track 0.00 -> 66.0 mm, vias 0 -> 3
- net Reset: track 0.00 -> 65.9 mm, vias 0 -> 1
- net GND: track 9.93 -> 69.8 mm, vias 8 -> 36
- net LED_G: track 0.00 -> 58.2 mm, vias 0 -> 1
- net Antenn_Digital_2: track 0.00 -> 58.0 mm
- net IR_T_OUTSIDE: track 0.00 -> 54.9 mm, vias 0 -> 2
- net Antenn_Digital_1: track 0.00 -> 54.0 mm
- net LED_B: track 0.00 -> 53.5 mm, vias 0 -> 1
- net IR_T_INSIDE: track 0.00 -> 50.4 mm
- net M_LOCK: track 0.00 -> 49.8 mm
- net BAT_MON: track 42.6 -> 92.1 mm, vias 0 -> 2
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