File: Hardware/Kicad/CAT FLAP/CatFlap_PCB/CatFlap_PCB/CatFlap_PCB.kicad_sch (KiCad schematic)
At the start: 53 parts, among them J1 Conn_01x08, J2 Conn_01x03, J3 ${ALTIUM_VALUE}, J4 Conn_01x03_Socket, J5 Conn_ARM_SWD_TagConnect_TC203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, J6 Conn_01x02, J7 Conn_01x06, J8 Conn_01x20, J9 Conn_01x20, M1 Motor_DC, Q1 NX3008CBKS, Q2 Q_PMOS_DGS, SW1 SW_Push, SW2 SW_Push, SW3 SW_Push, SW4 SW_Push, T1 NX3008NBKS, T2 NX3008NBKS, U2 DRV8837DSGR, U3 TPS62132

Commit message: Add files via upload
Parts:
- removed C26 (x2): 1u, Capacitor_SMD:C_0603_1608Metric, symbol Device:C_Small
- removed J5: Conn_ARM_SWD_TagConnect_TC2030-NL, Connector:Tag-Connect_TC2030-IDC-NL_2x03_P1.27mm_Vertical, symbol Connector:Conn_ARM_SWD_TagConnect_TC2030-NL
- removed J7: Conn_01x06, Connector_PinHeader_2.54mm:PinHeader_1x06_P2.54mm_Vertical, symbol Connector_Generic:Conn_01x06
- removed SW4: SW_Push, Button_Switch_SMD:SW_Push_1P1T_NO_Vertical_Wuerth_434133025816, symbol Switch:SW_Push
- added C26 (x2): 1u, Capacitor_SMD:C_0603_1608Metric, symbol Device:C_Small
- added J5: Conn_01x03, Connector_PinHeader_2.54mm:PinHeader_1x03_P2.54mm_Vertical, symbol Connector_Generic:Conn_01x03
- added R5 (x2): 0, Resistor_SMD:R_0603_1608Metric, symbol Device:R
- added R5 (x2): 6.8, Resistor_SMD:R_0603_1608Metric, symbol Device:R
- C26: footprint Capacitor_SMD:C_0603_1608Metric -> Capacitor_SMD:C_0805_2012Metric
- C26: footprint Capacitor_SMD:C_0603_1608Metric -> Capacitor_SMD:C_1210_3225Metric
- D1: footprint LED_RGB_CLX5E:LED_RGB_CLX6E -> LED_SMD:LED_RGB_PLCC-6
- D2: ulrbuy (none) -> https://se.farnell.com/kingbright/l-934f3c/infrared-emitter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
- J1: footprint (none) -> Connector_PinHeader_2.54mm:PinHeader_1x08_P2.54mm_Vertical
- J3: footprint Connector_JST:JST_XH_B2B-XH-A_1x02_P2.50mm_Vertical -> Battery:BatteryHolder_MPD_BH-18650-PC2
- JP2, JP3, JP4: footprint (none) -> Jumper:SolderJumper-3_P1.3mm_Bridged12_RoundedPad1.0x1.5mm
- L1: footprint (none) -> Inductor_SMD:L_Coilcraft_XxL4020; urlBUY (none) -> https://se.farnell.com/coilcraft/xfl4020-222mec/inductor-2-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
- R2: value 20 -> 22
- SW3: footprint Button_Switch_SMD:SW_Push_1P1T_NO_6x6mm_H9.5mm -> Button_Switch_SMD:SW_Push_1P1T_NO_Vertical_Wuerth_434133025816
- T1: footprint NX3008NBKS:SOT363 -> Package_TO_SOT_SMD:SOT-363_SC-70-6
Connections:
- net GP1 is gone; now on net M_SLEEP: J9.2 (Pin_2)
- net GP16 is gone; now on net Antenn_Digital_1: J8.20 (Pin_20)
- net GP17 is gone; now on net Antenn_Digital_2: J8.19 (Pin_19)
- net GP2 is gone; now on net LED_B: J9.4 (Pin_4)
- net GP27_A1 is gone; now on net IR_R_INSIDE: J8.9 (Pin_9)
- net GP3 is gone; now on net LED_G: J9.5 (Pin_5)
- net GP4 is gone; now on net LED_R: J9.6 (Pin_6)
- net GP5 is gone; now on net M_UNLOCK: J9.7 (Pin_7)
- net GP6 is gone; now on net M_LOCK: J9.9 (Pin_9)
- net GP7 is gone; now on net IR_T_OUTSIDE: J9.10 (Pin_10)
- net GP8 is gone; now on net IR_T_INSIDE: J9.11 (Pin_11)
- net RUN is gone; now on net Reset: J8.11 (Pin_11)
- net Antenn_Analog: now also J1.6 (Pin_6), J5.1 (Pin_1); no longer J1.3 (Pin_3)
- net BAT_MON: now also J5.3 (Pin_3); no longer J8.7 (Pin_7)
- net GND: now also C26.1, C26.1
- net GP27_A0: now also J5.2 (Pin_2)
- net IR_R_INSIDE: now also R5.2; no longer D4.2 (A)
- net IR_R_OUTSIDE: now also J8.7 (Pin_7), R5.2; no longer D5.2 (A)
- net VDD: now also C26.2, F1.2, J1.3 (Pin_3), Q2.3 (S); no longer J1.2 (Pin_2), J3.2 (V+), J6.1 (Pin_1), Q2.1 (D)
- net at U2.2 (OUT1): now also M1.2 (-); no longer M1.1 (+)
- net at U2.3 (OUT2): now also M1.1 (+); no longer M1.2 (-)
- net at D2.1 (K), R5.2: now also R5.2
- net at D2.2 (A), JP2.2 (C): now also C26.2
- net at R5.1, T1.6: now also R5.1
- net at D3.1 (K), R5.2: now also R5.2
- net at D3.2 (A), JP3.2 (C): now also C26.2
- net at R5.1, T1.3: now also R5.1
- net ADC_VREF renamed ADC_VREF_Antenn
- net ADC_VREF_Antenn: now also J1.2 (Pin_2)
- new net: D5.2 (A), R5.1
- new net: J3.2 (V+), J6.1 (Pin_1), Q2.1 (D)
- new net: D4.2 (A), R5.1
- no-connect marks 0 -> 12
Other:
- note removed: "Serial Wire Debug (SWD)"
- moved on the sheet: J1
