File: Hardware/Kicad/CAT FLAP/CatFlap_PCB/CatFlap_PCB.kicad_pcb (KiCad board)
At the start: 2 copper layers, 196 x 25 mm, 66 parts, among them J1 Conn_01x08, J2 Conn_01x03, J3 Battery pack, J4 Conn_01x03_Socket, J5 Conn_01x03, J6 Conn_01x02, J8 Conn_01x20, J9 Conn_01x20, M1 Motor_DC, Q1 NX3008CBKS, Q2 Q_PMOS_DGS, SW1 SW_Push, SW2 SW_Push, SW3 SW_Push, T1 NX3008NBKS, T2 NX3008NBKS, T3 NX3008NBKS, U1 LM358_DFN, U2 DRV8837DSGR, U3 TPS62132

Commit message: Add files via upload
Parts:
- added H1: MountingHole, MountingHole:MountingHole_5mm, F.Cu at (179.3, 83.2)
- added H2: MountingHole, MountingHole:MountingHole_5mm, F.Cu at (119.3, 83.2)
Routing:
- net BAT_MON: track 92.1 -> 108.2 mm, vias 2 -> 3
- net +3.3V: track 322.4 -> 320.8 mm
- net GND: track 70.5 -> 69.2 mm, vias 38 -> 171
- net Net-(U3-PG): track 10.3 -> 9.59 mm
Other:
- outline, holes or cut-outs redrawn
