File: Hardware/Kicad/CAT FLAP/CatFlap_PCB/CatFlap_PCB.kicad_pcb (KiCad board)
At the start: 2 copper layers, 196 x 25 mm, 68 parts, among them J1 Conn_01x08, J2 Conn_01x03, J3 Battery pack, J4 Conn_01x03_Socket, J5 Conn_01x03, J6 Conn_01x02, J8 Conn_01x20, J9 Conn_01x20, M1 Motor_DC, Q1 NX3008CBKS, Q2 Q_PMOS_DGS, SW1 SW_Push, SW2 SW_Push, SW3 SW_Push, T1 NX3008NBKS, T2 NX3008NBKS, T3 NX3008NBKS, U1 LM358_DFN, U2 DRV8837DSGR, U3 TPS62132

Commit message: Add files via upload
Parts:
- added C10: 100n, Capacitor_SMD:C_0603_1608Metric, F.Cu at (85.0, 81.1)
- added C16: 100n, Capacitor_SMD:C_0603_1608Metric, F.Cu at (85.0, 82.7)
- added C9: 1u, Capacitor_SMD:C_0603_1608Metric, F.Cu at (67.0, 80.8)
- added R14: 100k, Resistor_SMD:R_0603_1608Metric, F.Cu at (122.6, 91.5)
- added R22: 100k, Resistor_SMD:R_0603_1608Metric, F.Cu at (122.2, 94.5)
- added R23: 100k, Resistor_SMD:R_0603_1608Metric, F.Cu at (83.8, 85.0)
- added R24: 100k, Resistor_SMD:R_0603_1608Metric, F.Cu at (82.7, 80.2)
- added R25: 100k, Resistor_SMD:R_0603_1608Metric, F.Cu at (85.0, 79.5)
- added R26: 100k, Resistor_SMD:R_0603_1608Metric, F.Cu at (83.6, 91.6)
- U1: footprint Package_DFN_QFN:DFN-8-1EP_2x2mm_P0.5mm_EP1.05x1.75mm -> Package_SO:SOIC-8-1EP_3.9x4.9mm_P1.27mm_EP2.29x3mm
- moved C5 6.08 mm to (79.7, 90.4)
- moved R15 6.08 mm to (79.7, 92.0)
- moved R10 6.08 mm to (82.0, 91.2)
- moved R20 6.08 mm to (77.2, 91.2)
- moved U1 2.97 mm to (79.2, 85.2)
Connections:
- U1 pad 3: GND -> Net-(U1A-+)
- U1 pad 5: GND -> Net-(U1B-+)
Routing:
- net +3.3V: track 320.8 -> 345.6 mm, vias 5 -> 7
- net Net-(U1A-+): track 0.00 -> 10.8 mm
- net Net-(D4-A): track 15.2 -> 23.0 mm
- net Net-(U1B-+): track 0.00 -> 5.51 mm
- net IR_R_INSIDE: track 104.4 -> 109.5 mm
- net GND: track 69.2 -> 71.7 mm, vias 171 -> 162
- net Net-(U1A--): track 5.34 -> 7.10 mm
- net M_SLEEP: track 32.6 -> 31.0 mm
- net Net-(C6-Pad1): track 7.74 -> 9.18 mm
- net Net-(U1B--): track 10.7 -> 12.0 mm
- net Net-(J3-V+): track 178.3 -> 177.5 mm
- net M_LOCK: track 49.8 -> 50.6 mm
