File: Hardware/Kicad/CAT FLAP/CatFlap_PCB/CatFlap_PCB.kicad_sch (KiCad schematic)
At the start: 38 parts, among them J1 USB_C_Receptacle_USB2.0, J3 ${ALTIUM_VALUE}, J3 Conn_01x02_Socket, J5 Conn_ARM_SWD_TagConnect_TC203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, M1 Motor_DC, Q1 DMC2053UVT, T1 NX3008NBKS, T2 NX3008NBKS, U1 RP2040, U2 DRV8837DSGR, Y1 12MHz

Commit message: Add files via upload
Parts:
- added C26 (x2): 1u, Capacitor_SMD:C_0603_1608Metric, symbol Device:C_Small
- added D2, D3: IR-LED, Connector_PinHeader_2.54mm:PinHeader_1x02_P2.54mm_Horizontal, symbol Device:LED
- added D4, D5: LED, Connector_PinHeader_2.54mm:PinHeader_1x02_P2.54mm_Horizontal, symbol Device:LED
- added JP2, JP3: SolderJumper_3_Bridged12, symbol Jumper:SolderJumper_3_Bridged12
- added R5 (x2): 100, Resistor_SMD:R_0402_1005Metric, symbol Device:R
- added unit 2 of T2 (x2)
- added U3: TPS62132, Package_DFN_QFN:VQFN-16-1EP_3x3mm_P0.5mm_EP1.68x1.68mm_ThermalVias, symbol Regulator_Switching:TPS62132
- M1: footprint (none) -> Connector_PinHeader_2.54mm:PinHeader_1x02_P2.54mm_Horizontal
Connections:
- net +3V0: now also C26.2, C26.2, JP2.1 (A), JP3.1 (A)
- net GND: now also U2.9 (EXP), C26.1, C26.1, D4.1 (K), D5.1 (K), T2.4, T2.4, U3.15 (PGND), U3.16 (PGND), U3.17 (EP), U3.6 (AGND)
- net VDD: now also JP2.3 (B), JP3.3 (B)
- net D+ESD renamed USB_DP
- net D-ESD renamed USB_DM
- new net: R5.1, T2.3 (x2)
- new net: D2.1 (K), R5.2
- new net: D2.2 (A), JP2.2 (C)
- new net: D3.1 (K), R5.2
- new net: D3.2 (A), JP3.2 (C)
- new net: U3.1 (SW), U3.2 (SW), U3.3 (SW)
- new net: U3.11 (PVIN), U3.12 (PVIN)
- new net IR_R_IN: D4.2 (A)
- new net IR_R_OUT: D5.2 (A)
- new net IR_T_IN: T2.5
- new net IR_T_OUT: T2.5
Other:
- note added: "IR-SENSORS"
- note added: "RP2040"
- note added: "Receiver"
- note added: "Transmitter"
- moved on the sheet: C1, C10, C11, C2, C26, C3, C4, C5, C6, C7, C8, C9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

Commit message: Updated Powermanagement
Parts:
- removed C26: 100u, Capacitor_SMD:C_0603_1608Metric, symbol Device:C_Small
- removed J3: Conn_01x02_Socket, Connector_PinSocket_2.54mm:PinSocket_1x02_P2.54mm_Vertical, symbol Connector:Conn_01x02_Socket
- removed unit 2 of T2 (x2)
- added C26: 22u, Capacitor_SMD:C_0603_1608Metric, symbol Device:C_Small
- added C26: 100n, Capacitor_SMD:C_0603_1608Metric, symbol Device:C_Small
- added C26: 100u, Capacitor_SMD:C_0603_1608Metric, symbol Device:C_Small
- added C26: 10u, Capacitor_SMD:C_0603_1608Metric, symbol Device:C_Small
- added C26: 3.3n, Capacitor_SMD:C_0603_1608Metric, symbol Device:C_Small
- added J4: Conn_01x03_Socket, symbol Connector:Conn_01x03_Socket
- added JP4: SolderJumper_3_Bridged12, symbol Jumper:SolderJumper_3_Bridged12
- added L1: 2.2u, symbol Device:L
- added Q2: Q_PMOS_DGS, symbol Device:Q_PMOS_DGS
- added R5: 100k, Resistor_SMD:R_0402_1005Metric, symbol Device:R
- added T1: NX3008NBKS, NX3008NBKS:SOT363, symbol NX3008NBKS:NX3008NBKS
Connections:
- net +3V0: now also U3.14 (VOS), C26.2, JP4.1 (A), L1.2, R5.2; no longer U2.7 (~{SLEEP})
- net GND: now also U3.5 (FB), U3.7 (FSW), U3.8 (DEF), C26.1, C26.1, C26.1, C26.1, C26.2, Q2.2 (G), T1.1, T1.4
- net VBUS: now also J4.3 (Pin_3)
- net VDD: now also Q2.1 (D)
- net at R5.1: now also T1.6
- net at U3.1 (SW), U3.2 (SW), U3.3 (SW): now also L1.1
- net V_BAT: now reaches U3.10 (AVIN)
- net V_BAT: now also Q1.2 (S), R15.1, U3.11 (PVIN), U3.12 (PVIN), U3.13 (EN), C26.2, C26.2, J4.2 (Pin_2)
- net at U3.4 (PG): now also R5.1
- net at U3.9 (SS/TR): now also C26.1
- net at R5.1: now also T1.3
- net IR_R_IN renamed IR_R_INSIDE
- net IR_R_OUT renamed IR_R_OUTSIDE
- new net: JP4.2 (C), U2.7 (~{SLEEP})
- new net: C26.2, J4.1 (Pin_1), Q2.3 (S)
- new net IR_T_INSIDE: T1.2
- new net IR_T_OUTSIDE: T1.5
- new net M_SLEEP: JP4.3 (B)
Other:
- note removed: "Kolla hur AA batterier ska kopplas, decoupling etc"
- moved on the sheet: C1, C10, C11, C2, C26, C3, C4, C5, C6, C7, C8, C9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

Commit message: Add files via upload
Parts:
- removed JP1: SolderJumper_3_Bridged12, symbol Jumper:SolderJumper_3_Bridged12
- added F1: Polyfuse, Fuse:Fuse_1812_4532Metric, symbol Device:Polyfuse
- added J2: Conn_01x03, symbol Connector_Generic:Conn_01x03
- added J6: Conn_01x02, symbol Connector_Generic:Conn_01x02
- added J7: Conn_01x06, Connector_PinHeader_2.54mm:PinHeader_1x06_P2.54mm_Vertical, symbol Connector_Generic:Conn_01x06
- added J8, J9: Conn_01x20, Connector_PinHeader_2.54mm:PinHeader_1x20_P2.54mm_Vertical, symbol Connector_Generic:Conn_01x20
- added SW1, SW2: SW_Push, Button_Switch_THT:SW_PUSH_6mm_H4.3mm, symbol Switch:SW_Push
- added SW3: SW_Push, Button_Switch_SMD:SW_Push_1P1T_NO_6x6mm_H9.5mm, symbol Switch:SW_Push
- added SW4: SW_Push, Button_Switch_SMD:SW_Push_1P1T_NO_Vertical_Wuerth_434133025816, symbol Switch:SW_Push
- Q1: value DMC2053UVT -> NX3008CBKS; FDC6321C Datasheet https://4donline.ihs.com/images/VipMasterIC/IC/ONSM/ONSM-S-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 -> (none); URLBUY (none) -> https://se.farnell.com/nexperia/nx3008cbks-115/mosfet-n-p-c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; URLbuy https://se.farnell.com/on-semiconductor/fdc6321c/mosfet-dua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 -> (none)
- Q1: value DMC2053UVT -> NX3008CBKS; URLBUY (none) -> https://se.farnell.com/nexperia/nx3008cbks-115/mosfet-n-p-c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
- Q2: footprint (none) -> Package_TO_SOT_SMD:SOT-23; URLBUY (none) -> https://se.farnell.com/multicomp-pro/cdm2319ds/mosfet-p-ch-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
- R1, R13, R14, R15, R17, R2, R3, R4, R5: footprint Resistor_SMD:R_0402_1005Metric -> Resistor_SMD:R_0603_1608Metric
- R10: footprint (none) -> Resistor_SMD:R_0603_1608Metric
- T1: footprint NX3008NBKS:SOT363 -> Package_TO_SOT_SMD:SOT-363_SC-70-6
- T1: footprint NX3008NBKS:SOT363 -> Package_TO_SOT_SMD:SOT-363_SC-70-6; URLbuy (none) -> https://se.farnell.com/nexperia/nx3008nbks-115/mosfet-nn-ch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
- U2: Purchase-URL https://www.snapeda.com/api/url_track_click_mouser/?unipart_id=230051&manufacturer=Texas Instruments&part_name=DRV8837DSGR&search_term=drv8837dsgr -> https://www.snapeda.com/api/url_track_click_mouser/?unipart_id=230051&manufacturer=Texas https://se.farnell.com/texas-instruments/drv8837dsgr/motor-driver-dc-brushed-1-8a-wson/dp/3005855?st=drv8837dsgr
- U3: URLBUY (none) -> https://se.farnell.com/texas-instruments/tps62132rgtr/dc-dc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
Connections:
- net +3V0 is gone; now on net +3.3V: C26.2, C26.2, C26.2, C26.2, D1.4 (BA), D1.5 (GA), D1.6 (RA), JP2.1 (A), JP3.1 (A), JP4.1 (A), L1.2, R5.2, U2.8 (VCC), U3.14 (VOS)
- net +3.3V: now also J2.3 (Pin_3), J7.6 (Pin_6)
- net BAT_MON_EN: now also Q1.2 (G); no longer Q1.1 (G)
- net Earth: now also SW1.1, SW2.1, SW3.1, SW4.1; no longer C1.2, C10.2, C11.2, C2.2, C3.2, C4.2, C5.2, C6.2, C7.2, C8.1, C9.2, U1.19 (TESTEN), U1.57 (GND)
- net GND: now also C1.2, C10.2, C11.2, C2.2, C3.2, C4.2, C5.2, C6.2, C7.2, C8.1, C9.2, Q1.1 (S), U1.19 (TESTEN), U1.57 (GND), J6.2 (Pin_2), J7.1 (Pin_1), J8.13 (Pin_13), J8.18 (Pin_18), J8.3 (Pin_3), J9.13 (Pin_13), J9.18 (Pin_18), J9.3 (Pin_3), J9.8 (Pin_8); no longer Q1.5 (S)
- net Reset: now also J7.5 (Pin_5), SW3.2
- net SWDCLK: now also J7.3 (Pin_3)
- net SWDIO: now also J7.2 (Pin_2)
- net VBUS: now also J8.1 (Pin_1)
- net VDD: now also J2.1 (Pin_1), J6.1 (Pin_1)
- net V_BAT: now also Q1.4 (S); no longer Q1.2 (S)
- net at C26.2, C26.2, U2.1 (VM): now also J2.2 (Pin_2)
- net at Q1.6 (D), R15.2: now also Q1.5 (G); no longer Q1.3 (G)
- net SWO: now reaches J5.6 (SWO)
- net SWO: now also J7.4 (Pin_4)
- net at C26.2, Q2.3 (S): now also F1.2; no longer J4.1 (Pin_1)
- net at R13.1: now also Q1.3 (D); no longer Q1.4 (D)
- new net: F1.1, J4.1 (Pin_1)
- new net 3V3: J8.5 (Pin_5)
- new net 3V3_EN: J8.4 (Pin_4)
- new net ADC_VREF: J8.6 (Pin_6)
- new net AGND: J8.8 (Pin_8)
- new net Bootsel: SW4.2
- new net Cat+: SW2.2
- new net GP0: J9.1 (Pin_1)
- new net GP1: J9.2 (Pin_2)
- new net GP10: J9.14 (Pin_14)
- new net GP11: J9.15 (Pin_15)
- new net GP12: J9.16 (Pin_16)
- new net GP13: J9.17 (Pin_17)
- new net GP14: J9.19 (Pin_19)
- new net GP15: J9.20 (Pin_20)
- new net GP16: J8.20 (Pin_20)
- new net GP17: J8.19 (Pin_19)
- new net GP18: J8.17 (Pin_17)
- new net GP19: J8.16 (Pin_16)
- new net GP2: J9.4 (Pin_4)
- new net GP20: J8.15 (Pin_15)
- new net GP21: J8.14 (Pin_14)
- new net GP22: J8.12 (Pin_12)
- new net GP27_A0: J8.10 (Pin_10)
- new net GP27_A1: J8.9 (Pin_9)
- new net GP28_A2: J8.7 (Pin_7)
- new net GP3: J9.5 (Pin_5)
- new net GP4: J9.6 (Pin_6)
- new net GP5: J9.7 (Pin_7)
- new net GP6: J9.9 (Pin_9)
- new net GP7: J9.10 (Pin_10)
- new net GP8: J9.11 (Pin_11)
- new net GP9: J9.12 (Pin_12)
- new net Gear: SW1.2
- new net RUN: J8.11 (Pin_11)
- new net VSYS: J8.2 (Pin_2)
- no-connect marks 34 -> 39
Other:
- note added: "Buttons"
- note added: "Pins for Raspberry Pi"
- moved on the sheet: C1, C10, C11, C2, C26, C3, C4, C5, C6, C7, C8, C9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

Commit message: Add files via upload
Parts:
- removed C1, C10, C2, C3, C4, C5, C9: 100nF, symbol Device:C
- removed C11, C8: 2.2uF, symbol Device:C
- removed C26 (x2): 1u, Capacitor_SMD:C_0603_1608Metric, symbol Device:C_Small
- removed C6, C7: 15pF, symbol Device:C
- removed J1: USB_C_Receptacle_USB2.0, USB_C_Rece:USB_C_Receptacle_JAE_DX07S016JA1R1500-V4, symbol Connector:USB_C_Receptacle_USB2.0
- removed J5: Conn_ARM_SWD_TagConnect_TC2030-NL, Connector:Tag-Connect_TC2030-IDC-NL_2x03_P1.27mm_Vertical, symbol Connector:Conn_ARM_SWD_TagConnect_TC2030-NL
- removed J7: Conn_01x06, Connector_PinHeader_2.54mm:PinHeader_1x06_P2.54mm_Vertical, symbol Connector_Generic:Conn_01x06
- removed R10: 1k, Resistor_SMD:R_0603_1608Metric, symbol Device:R
- removed R3, R4: 5k1, Resistor_SMD:R_0603_1608Metric, symbol Device:R
- removed SW4: SW_Push, Button_Switch_SMD:SW_Push_1P1T_NO_Vertical_Wuerth_434133025816, symbol Switch:SW_Push
- removed U1: RP2040, Package_DFN_QFN:QFN-56-1EP_7x7mm_P0.4mm_EP3.2x3.2mm, symbol MCU_RaspberryPi:RP2040
- removed Y1: 12MHz, symbol Device:Crystal_GND23
- added C26 (x2): 1u, Capacitor_SMD:C_0603_1608Metric, symbol Device:C_Small
- added C26 (x4): 1.4p, Capacitor_SMD:C_0603_1608Metric, symbol Device:C_Small
- added C26 (x2): 100n, Capacitor_SMD:C_0603_1608Metric, symbol Device:C_Small
- added J1: Conn_01x08, Connector_PinHeader_2.54mm:PinHeader_1x08_P2.54mm_Vertical, symbol Connector_Generic:Conn_01x08
- added J5: Conn_01x03, Connector_PinHeader_2.54mm:PinHeader_1x03_P2.54mm_Vertical, symbol Connector_Generic:Conn_01x03
- added R5 (x6): 0, Resistor_SMD:R_0603_1608Metric, symbol Device:R
- added R5 (x2): 6.8, Resistor_SMD:R_0603_1608Metric, symbol Device:R
- added R5 (x2): 100k, Resistor_SMD:R_0603_1608Metric, symbol Device:R
- added U1: LM358_DFN, Package_DFN_QFN:DFN-8-1EP_2x2mm_P0.5mm_EP1.05x1.75mm, symbol Amplifier_Operational:LM358_DFN
- C26: footprint Capacitor_SMD:C_0603_1608Metric -> Capacitor_SMD:C_0805_2012Metric
- C26: footprint Capacitor_SMD:C_0603_1608Metric -> Capacitor_SMD:C_1210_3225Metric
- D1: footprint LED_RGB_CLX5E:LED_RGB_CLX6E -> LED_SMD:LED_RGB_PLCC-6
- D2: ulrbuy (none) -> https://se.farnell.com/kingbright/l-934f3c/infrared-emitter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
- J2, J4: footprint (none) -> Connector_PinHeader_2.54mm:PinHeader_1x03_P2.54mm_Vertical
- J3: footprint Connector_JST:JST_XH_B2B-XH-A_1x02_P2.50mm_Vertical -> Battery:BatteryHolder_MPD_BH-18650-PC2
- J6: footprint (none) -> Connector_PinHeader_2.54mm:PinHeader_1x02_P2.54mm_Vertical
- JP2, JP3, JP4: footprint (none) -> Jumper:SolderJumper-3_P1.3mm_Bridged12_RoundedPad1.0x1.5mm
- L1: footprint (none) -> Inductor_SMD:L_Coilcraft_XxL4020; urlBUY (none) -> https://se.farnell.com/coilcraft/xfl4020-222mec/inductor-2-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
- R2: value 20 -> 22
- R5: value 100 -> 6.8
- SW3: footprint Button_Switch_SMD:SW_Push_1P1T_NO_6x6mm_H9.5mm -> Button_Switch_SMD:SW_Push_1P1T_NO_Vertical_Wuerth_434133025816
- T1: footprint NX3008NBKS:SOT363 -> Package_TO_SOT_SMD:SOT-363_SC-70-6
Connections:
- net AGND is gone; now on net GND: J8.8 (Pin_8)
- net Earth is gone; now on net GND: SW1.1, SW2.1, SW3.1
- net GP0 is gone; now on net Gear: J9.1 (Pin_1)
- net GP1 is gone; now on net M_SLEEP: J9.2 (Pin_2)
- net GP15 is gone; now on net Cat+: J9.20 (Pin_20)
- net GP2 is gone; now on net LED_B: J9.4 (Pin_4)
- net GP22 is gone; now on net BAT_MON_EN: J8.12 (Pin_12)
- net GP27_A1 is gone; now on net IR_R_INSIDE: J8.9 (Pin_9)
- net GP28_A2 is gone; now on net IR_R_OUTSIDE: J8.7 (Pin_7)
- net GP3 is gone; now on net LED_G: J9.5 (Pin_5)
- net GP4 is gone; now on net LED_R: J9.6 (Pin_6)
- net GP5 is gone; now on net M_UNLOCK: J9.7 (Pin_7)
- net GP6 is gone; now on net M_LOCK: J9.9 (Pin_9)
- net GP7 is gone; now on net IR_T_OUTSIDE: J9.10 (Pin_10)
- net GP8 is gone; now on net IR_T_INSIDE: J9.11 (Pin_11)
- net RUN is gone; now on net Reset: J8.11 (Pin_11)
- net VSYS is gone; now on net +3.3V: J8.2 (Pin_2)
- net +3.3V: now also D4.1 (K), D5.1 (K), C26.2, C26.2, C26.2, J1.1 (Pin_1), U1.8 (V+)
- net BAT_MON: now also J5.3 (Pin_3)
- net GND: now also C26.1, C26.1, C26.1, C26.1, J1.7 (Pin_7), J1.8 (Pin_8), R5.2, R5.2, U1.3 (+), U1.4 (V-), U1.5 (+), U1.9 (PAD); no longer D4.1 (K), D5.1 (K)
- net GP27_A0: now also J5.2 (Pin_2)
- net IR_R_INSIDE: now also R5.1, R5.1; no longer D4.2 (A)
- net IR_R_OUTSIDE: now also R5.1, R5.1; no longer D5.2 (A)
- net VBUS: now also C26.2
- net VDD: now also C26.2, F1.2, Q2.3 (S), J1.3 (Pin_3); no longer J3.2 (V+), J6.1 (Pin_1), Q2.1 (D)
- net at U2.2 (OUT1): now also M1.2 (-); no longer M1.1 (+)
- net at U2.3 (OUT2): now also M1.1 (+); no longer M1.2 (-)
- net at D2.1 (K), R5.2: now also R5.2
- net at D2.2 (A), JP2.2 (C): now also C26.2
- net at R5.1, T1.6: now also R5.1
- net at D3.1 (K), R5.2: now also R5.2
- net at D3.2 (A), JP3.2 (C): now also C26.2
- net at R5.1, T1.3: now also R5.1
- net ADC_VREF renamed ADC_VREF_Antenn
- net ADC_VREF_Antenn: now also J1.2 (Pin_2)
- net GP16 renamed Antenn_Digital_1
- net Antenn_Digital_1: now also J1.4 (Pin_4)
- net GP17 renamed Antenn_Digital_2
- net Antenn_Digital_2: now also J1.5 (Pin_5)
- new net: C26.2, R5.1, R5.2, U1.2 (-)
- new net: C26.1, D4.2 (A), R5.2
- new net: C26.1, R5.1, R5.2, U1.1
- new net: C26.1, D5.2 (A), R5.2
- new net: J3.2 (V+), J6.1 (Pin_1), Q2.1 (D)
- new net: C26.1, R5.1, R5.2, U1.7
- new net: C26.2, R5.1, R5.2, U1.6 (-)
- new net Antenn_Analog: J1.6 (Pin_6), J5.1 (Pin_1)
- no-connect marks 39 -> 12
Other:
- note added: "Antenna"
- note added: "POWERFLAGS"
- note removed: "RP2040"
- note removed: "RP2040 decoupling"
- note removed: "Serial Wire Debug (SWD)"
- note removed: "USB-C"
- moved on the sheet: C26, D1, D2, D3, F1, J2, J3, J4, J6, J8, J9, JP2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

Commit message: Add files via upload
Parts:
- added H1, H2: MountingHole, MountingHole:MountingHole_5mm, symbol Mechanical:MountingHole
Other:
- note added: "Mounting Hole"
Changed lines of the file:
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@@
+    (fill (type none))
+  )
+  (rectangle (start 106.045 175.895) (end 156.845 192.405)
+    (stroke (width 0) (type default))
     (fill (type none))
   )
@@
     (effects (font (size 1.27 1.27)) (justify left bottom))
   )
+  (text "Mounting Hole" (at 106.045 181.61 0)
+    (effects (font (size 4 4)) (justify left bottom))
+  )
   (text "POWER MANAGEMENT" (at 200.66 85.725 0)
     (effects (font (size 4 4)) (justify left bottom))
@@
     )
   )
+  (symbol (lib_id "Mechanical:MountingHole") (at 113.665 186.69 0) (unit 1)
+    (in_bom yes) (on_board yes) (dnp no) (fields_autoplaced)
+    (property "Reference" "H1" (at 116.84 185.42 0)
+      (effects (font (size 1.27 1.27)) (justify left))
+    )
+    (property "Value" "MountingHole" (at 116.84 187.96 0)
+      (effects (font (size 1.27 1.27)) (justify left))
+    )
+    (property "Footprint" "MountingHole:MountingHole_5mm" (at 113.665 186.69 0)
+      (effects (font (size 1.27 1.27)) hide)
+    )
+    (property "Datasheet" "~" (at 113.665 186.69 0)
+      (effects (font (size 1.27 1.27)) hide)
+    )
+    (instances
+      (project "CatFlap_PCB"
+        (path "/bddc0924-0264-4c85-82d9-54676452eec2"
+          (reference "H1") (unit 1)
+        )
+      )
+    )
+  )
   (symbol (lib_id "Connector:Conn_01x03_Socket") (at 220.98 93.98 0) (mirror y) (unit 1)
     (in_bom yes) (on_board yes) (dnp no)
@@
         )
       )
+    )
+  )
+  (symbol (lib_id "Mechanical:MountingHole") (at 135.255 186.69 0) (unit 1)
+    (in_bom yes) (on_board yes) (dnp no) (fields_autoplaced)
+    (property "Reference" "H2" (at 138.43 185.42 0)
+      (effects (font (size 1.27 1.27)) (justify left))
+    )
+    (property "Value" "MountingHole" (at 138.43 187.96 0)
+      (effects (font (size 1.27 1.27)) (justify left))
+    )
+    (property "Footprint" "MountingHole:MountingHole_5mm" (at 135.255 186.69 0)
+      (effects (font (size 1.27 1.27)) hide)
+    )
+    (property "Datasheet" "~" (at 135.255 186.69 0)
+      (effects (font (size 1.27 1.27)) hide)
+    )
+    (instances
+      (project "CatFlap_PCB"
+        (path "/bddc0924-0264-4c85-82d9-54676452eec2"
+          (reference "H2") (unit 1)
+        )
+      )

Commit message: Add files via upload
Parts:
- added C26 (x2): 100n, Capacitor_SMD:C_0603_1608Metric, symbol Device:C_Small
- added C26: 1u, Capacitor_SMD:C_0603_1608Metric, symbol Device:C_Small
- added R5 (x6): 100k, Resistor_SMD:R_0603_1608Metric, symbol Device:R
- U1: footprint Package_DFN_QFN:DFN-8-1EP_2x2mm_P0.5mm_EP1.05x1.75mm -> Package_SO:SOIC-8-1EP_3.9x4.9mm_P1.27mm_EP2.29x3mm
Connections:
- net +3.3V: now also C26.2, C26.2, C26.2, R5.1, R5.1
- net GND: now also C26.1, C26.1, C26.1, R5.1, R5.1, R5.2, R5.2; no longer U1.3 (+), U1.5 (+)
- net M_LOCK: now also R5.1
- net M_UNLOCK: now also R5.2
- new net: R5.2, R5.2, U1.3 (+)
- new net: R5.1, R5.2, U1.5 (+)
Other:
- moved on the sheet: C26, D5, J3, J6, JP4, R5, U1B
